Commit message: init kp kd

File: src/mjlab/asset_zoo/robots/x3/x3.urdf (robot description, URDF)
Before this commit: robot X03B, 30 links, 29 joints
Links:
- link left_knee_link: mass 0.8 -> 0.6
- link right_knee_link: mass 0.8 -> 0.6
Joints:
- joint left_ankle_pitch_joint: origin xyz=0 0 -0.45 rpy=0 0 0 -> xyz=0 0 -0.39 rpy=0 0 0
- joint right_ankle_pitch_joint: origin xyz=0 0 -0.45 rpy=0 0 0 -> xyz=0 0 -0.39 rpy=0 0 0
- joint right_hip_pitch_joint: origin xyz=0 -0.0495 0 rpy=0 -0.00824 0 -> xyz=0 -0.0495 0 rpy=0 0 0
